File: Hardware/PCB/Hornbill Open Universal Remote.kicad_pcb (KiCad board)
At the start: 2 copper layers, 93 x 60 mm, 75 parts, among them CON1 USB-MINI-B, M1 ESP-WROOM-32, P1 CONN_01X14, P10 CONN_01X14, P11 CONN_01X14, P12 CONN_01X14, P13 CONN_01X14, P14 CONN_01X14, P15 CONN_01X14, P16 CONN_01X02, P17 CONN_01X03, P18 CONN_01X03, P19 CONN_01X03, P2 CONN_01X03, P20 CONN_01X01, P21 CONN_01X02, P22 CONN_01X02, P23 CONN_01X06, P24 CONN_01X02, P25 CONN_01X02, P26 CONN_01X02, P3 CONN_01X14, P4 CONN_01X14, P5 CONN_01X14, P6 CONN_01X14, P7 CONN_01X14, P8 CONN_01X14, P9 CONN_01X14, Q2 Q_NPN_BEC, Q3 S8050, Q4 S8050, SW1 SW_PUSH, SW2 SW_PUSH, U1 AP2112K, U2 OSH_Symbol, U3 EE_Logo, U4 EE_Logo, U5 MountingHole, U6 MountingHole, U7 MountingHole, U8 MountingHole, U9 CP2102, Y1 32.768KHz RTC Crystal

Commit message: Legend modified and gerber file generated
Other:
- board text added: "10"
- board text added: "11"
- board text added: "12"
- board text added: "14"
- board text added: "18"
- board text added: "19"
- board text added: "2"
- board text added: "22"
- board text added: "23"
- board text added: "25"
- board text added: "26"
- board text added: "27"
- board text added: "34"
- board text added: "35"
- board text added: "4"
- board text added: "5"
- board text added: "7"
- board text added: "8"
- board text added: "9"
- board text removed: "IO10"
- board text removed: "IO11"
- board text removed: "IO12"
- board text removed: "IO14"
- board text removed: "IO18"
- board text removed: "IO19"
- board text removed: "IO2"
- board text removed: "IO22"
- board text removed: "IO23"
- board text removed: "IO25"
- board text removed: "IO26"
- board text removed: "IO27"
- board text removed: "IO34"
- board text removed: "IO35"
- board text removed: "IO4"
- board text removed: "IO5"
- board text removed: "IO7"
- board text removed: "IO8"
- board text removed: "IO9"
Changed lines of the file:
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@@
     (links 108)
     (no_connects 0)
-    (area 64.924999 67.424999 158.075001 127.575001)
+    (area 34.650002 52.3 165.100001 140.100001)
     (thickness 1.6)
     (drawings 61)
@@
   (module Explore:cp2102_xl2 (layer F.Cu)
     (at 140.97 101.854 180)
-    (fp_text reference U9 (at -0.24892 -6.49986 180) (layer F.SilkS) hide
-      (effects (font (thickness 0.3048)))
+    (fp_text reference U9 (at 3.302 -2.794 180) (layer F.SilkS)
+      (effects (font (size 0.6 0.6) (thickness 0.15)))
     )
     (fp_text value CP2102 (at 0.24892 6.49986 180) (layer F.SilkS) hide
@@
     (effects (font (size 1.016 1.016) (thickness 0.254)) (justify mirror))
   )
-  (gr_text IO18 (at 112.522 73.152 90) (layer F.SilkS)
+  (gr_text 18 (at 112.522 72.644 90) (layer F.SilkS)
     (effects (font (size 1.016 1.016) (thickness 0.254)))
   )
-  (gr_text IO14 (at 109.728 73.152 90) (layer F.SilkS)
+  (gr_text 14 (at 109.728 72.644 90) (layer F.SilkS)
     (effects (font (size 1.016 1.016) (thickness 0.254)))
   )
-  (gr_text IO12 (at 107.315 73.152 90) (layer F.SilkS)
+  (gr_text 12 (at 107.188 72.644 90) (layer F.SilkS)
     (effects (font (size 1.016 1.016) (thickness 0.254)))
   )
-  (gr_text IO5 (at 104.648 72.644 90) (layer F.SilkS)
+  (gr_text 5 (at 104.648 72.644 90) (layer F.SilkS)
     (effects (font (size 1.016 1.016) (thickness 0.254)))
   )
-  (gr_text IO2 (at 102.362 72.644 90) (layer F.SilkS)
+  (gr_text 2 (at 102.362 72.644 90) (layer F.SilkS)
     (effects (font (size 1.016 1.016) (thickness 0.254)))
   )
-  (gr_text IO4 (at 99.822 72.644 90) (layer F.SilkS)
+  (gr_text 4 (at 99.822 72.644 90) (layer F.SilkS)
     (effects (font (size 1.016 1.016) (thickness 0.254)))
   )
-  (gr_text IO7 (at 97.155 72.771 90) (layer F.SilkS)
+  (gr_text 7 (at 97.155 72.771 90) (layer F.SilkS)
     (effects (font (size 1.016 1.016) (thickness 0.254)))
   )
-  (gr_text IO9 (at 92.202 72.771 90) (layer F.SilkS)
+  (gr_text 9 (at 92.202 72.771 90) (layer F.SilkS)
     (effects (font (size 1.016 1.016) (thickness 0.254)))
   )
-  (gr_text IO8 (at 94.488 72.771 90) (layer F.SilkS)
+  (gr_text 8 (at 94.488 72.771 90) (layer F.SilkS)
     (effects (font (size 1.016 1.016) (thickness 0.254)))
   )
-  (gr_text IO10 (at 89.408 72.898 90) (layer F.SilkS)
+  (gr_text "10\n" (at 89.408 72.898 90) (layer F.SilkS)
     (effects (font (size 1.016 1.016) (thickness 0.254)))
   )
-  (gr_text IO11 (at 86.995 72.898 90) (layer F.SilkS)
+  (gr_text 11 (at 86.995 72.898 90) (layer F.SilkS)
     (effects (font (size 1.016 1.016) (thickness 0.254)))
   )
@@
     (effects (font (size 1.016 1.016) (thickness 0.254)))
   )
-  (gr_text "IO35\n" (at 114.935 122.555 90) (layer F.SilkS)
+  (gr_text 35 (at 114.935 122.555 90) (layer F.SilkS)
     (effects (font (size 1.016 1.016) (thickness 0.254)))
   )
-  (gr_text "IO34\n" (at 112.395 122.555 90) (layer F.SilkS)
+  (gr_text 34 (at 112.395 122.555 90) (layer F.SilkS)
     (effects (font (size 1.016 1.016) (thickness 0.254)))
   )
-  (gr_text "IO27\n" (at 109.855 122.555 90) (layer F.SilkS)
+  (gr_text 27 (at 109.855 122.555 90) (layer F.SilkS)
     (effects (font (size 1.016 1.016) (thickness 0.254)))
   )
-  (gr_text "IO26\n" (at 107.442 122.555 90) (layer F.SilkS)
+  (gr_text 26 (at 107.442 122.555 90) (layer F.SilkS)
     (effects (font (size 1.016 1.016) (thickness 0.254)))
   )
-  (gr_text "IO25\n" (at 104.775 122.555 90) (layer F.SilkS)
+  (gr_text 25 (at 104.775 122.555 90) (layer F.SilkS)
     (effects (font (size 1.016 1.016) (thickness 0.254)))
   )
-  (gr_text "IO23\n" (at 102.235 122.555 90) (layer F.SilkS)
+  (gr_text 23 (at 102.235 122.555 90) (layer F.SilkS)
     (effects (font (size 1.016 1.016) (thickness 0.254)))
   )
-  (gr_text "IO22\n" (at 99.695 122.555 90) (layer F.SilkS)
+  (gr_text 22 (at 99.695 122.555 90) (layer F.SilkS)
     (effects (font (size 1.016 1.016) (thickness 0.254)))
   )
-  (gr_text IO19 (at 97.155 122.555 90) (layer F.SilkS)
+  (gr_text 19 (at 97.155 122.555 90) (layer F.SilkS)
     (effects (font (size 1.016 1.016) (thickness 0.254)))
   )
